Commit message: Separate original and adapted DexPilot

File: dex_retargeting/assets/robots/hands/leap_hand/leap_hand_right.urdf (robot description, URDF)
Before this commit: robot leap_right, 27 links, 26 joints
Links:
- removed link index_forward
- removed link thumb_forward
- added link index_normal
- added link middle_normal
- added link middle_side
- added link thumb_normal
Joints:
- removed joint index_forward_joint
- removed joint thumb_forward_joint
- added joint index_normal_joint: type fixed, parent index_tip_head, child index_normal, origin xyz=0.1 0 0 rpy=0 0 0
- added joint middle_normal_joint: type fixed, parent middle_tip_head, child middle_normal, origin xyz=0.1 0 0 rpy=0 0 0
- added joint middle_side_joint: type fixed, parent middle_tip_head, child middle_side, origin xyz=0 0 0.1 rpy=0 0 0
- added joint thumb_normal_joint: type fixed, parent thumb_tip_head, child thumb_normal, origin xyz=0.1 0 0 rpy=0 0 0
